Commit message: Add camera to URDF

File: jackal_description_cdt/urdf/jackal.urdf.xacro (robot description, xacro)
@@ -19,4 +19,5 @@
    <!--  Import modules for the EXTRM platform  -->
   <xacro:include filename="$(find jackal_description_cdt)/urdf/rooster.xacro"/>
+  <xacro:include filename="$(find jackal_description_cdt)/urdf/camera/base_camera.xacro"/>
   <xacro:macro name="wheel" params="prefix *joint_pose">
     <link name="${prefix}_wheel_link">
@@ -234,4 +235,7 @@
                  lidar="true"
                  simulation="true"/>
+  <xacro:base_camera name="camera"
+                     parent="base_link"
+                     simulation="true"/>
   <!-- Optional custom includes. -->
   <xacro:include filename="$(optenv JACKAL_URDF_EXTRAS empty.urdf)" />

File: jackal_description_cdt/urdf/rooster.xacro (robot description, xacro)
@@ -8,14 +8,14 @@
     <xacro:include filename="$(find jackal_description_cdt)/urdf/lidar/base_lidar.xacro"/>
     <!-- Properties -->
-    <xacro:property name="box_width" value="0.20" />
-    <xacro:property name="box_depth" value="0.17"/>
-    <xacro:property name="box_height" value="0.13" />
-    <!--
+    <xacro:property name="cylinder_height" value="0.30" />
+    <xacro:property name="cylinder_radius" value="0.04" />
     <link name="${name}">
       <visual>
         <geometry>
-          <box size="${box_width} ${box_depth} ${box_height}"/>
-        </geometry>
-        <material name="white"/>
+        <cylinder length="${cylinder_height}" radius="${cylinder_radius}"/>
+      </geometry>
+        <material name="white">
+          <color rgba="0.5 0.5 .5 1"/>
+        </material>
       </visual>
     </link>
@@ -23,7 +23,6 @@
       <parent link="base_link"/>
       <child link="${name}"/>
-      <origin xyz="0.05 0.0 ${box_height/2 + 0.15}" rpy="0 0 ${PI/2}"/>
+      <origin xyz="0.15 0.0 ${cylinder_height/2}" rpy="0 0 0"/>
     </joint>
-    -->
     <!-- LIDAR -->
     <xacro:if value="${lidar}">
@@ -34,5 +33,5 @@
                         translateX="0"
                         translateY="0"
-                        translateZ="${box_height/2}"
+                        translateZ="${cylinder_height/2}"
                         roll="0"
                         pitch="0"
