Commit message: Release 2021

File: jackal_description_cdt/urdf/lidar/base_lidar.xacro (robot description, xacro)
@@ -11,5 +11,5 @@
   <!-- param gpu_:  substring for hardware accelearation. (default: empty "", otherwise "gpu_")-->
   <xacro:property name="min_range" value="0.5"/>
-  <xacro:property name="max_range" value="50.0"/> <!-- was 120 -->
+  <!-- xacro:property name="max_range" value="50.0"/> <!- was 120 -->
   <xacro:property name="min_angle" value="-${PI}"/>
   <xacro:property name="max_angle" value="${PI}"/>
@@ -47,5 +47,5 @@
             <range>
               <min>${collision_range}</min>
-              <max>${max_range+1}</max>
+              <max>${max_range}</max>
               <resolution>0.001</resolution>
             </range>

File: jackal_description_cdt/urdf/rooster.xacro (robot description, xacro)
@@ -29,5 +29,5 @@
       <xacro:base_lidar name="horizontal"
                         parent="${name}"
-                        max_range="10"
+                        max_range="5"
                         min_range="0.1"
                         translateX="0"
